File: Placa_control/base.sch (EAGLE design)
At the start: 67 parts, among them Q10 IRF740, Q11 IRF740, Q5 IRF740, Q6 IRF740, Q7 IRF740, Q8 IRF740, Q9 IRF740

Commit message: Actualizacion de la placa y codigo demo
Parts:
- added C1: (no value), rcl:C-US025-030X050
- added C2: (no value), rcl:CPOL-USE2.5-5
- added IC1: MAX7219CNG, maxim:MAX7219CNG
- added JP1: (no value), pinhead:PINHD-1X3
- added M1: ARDUINO-NANO-3.0, diy-modules:ARDUINO-NANO-3.0
- added R46: 10k, rcl:R-US_0207/10
Connections:
- new net CLK: IC1.CLK, M1.D13/SCK
- new net CS: IC1.LOAD, M1.D12/MISO
- new net MOSI: IC1.DIN, M1.D11/MOSI
- new net N$15: IC1.ISET, R46.2
- new net N$21: JP1.1, M1.VIN
- new net V_LOGIC: JP1.2, X1-2.KL
- net 5V: now also C1.1, C2.+, IC1.VCC, JP1.3, M1.5V, R46.1; no longer X1-2.KL
- net A_IN: now also IC1.SEGA
- net B_IN: now also IC1.SEGB
- net C_IN: now also IC1.SEGC
- net D_IN: now also IC1.SEGD
- net EN_1_IN: now also IC1.DIG0
- net EN_2_IN: now also IC1.DIG1
- net EN_3_IN: now also IC1.DIG2
- net EN_4_IN: now also IC1.DIG3
- net E_IN: now also IC1.SEGE
- net F_IN: now also IC1.SEGF
- net GND: now also C1.2, C2.-, IC1.GND@1, IC1.GND@2, M1.GND.1, M1.GND.2
- net G_IN: now also IC1.SEGG
Other:
- note added: "Alimentación"
- note added: "Arduino NANO"
- note added: "Driver_LED"
- note added: "Salidas a displays"
- note added: "Selector de display"
- note added: "Selector de segmentos (A2G)"
- moved on the sheet: JP_ENABLE, JP_SEGMENTO, Q1, Q10, Q11, Q2, Q3, Q4, Q5, Q6, Q7, Q8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
